File: Third version prototype/PCB/Signal Processing/Signal_processing.brd (EAGLE design)
At the start: 75 x 36 mm, 140 parts, among them IC1 AD8066, IC2 ADG701BRTZN, IC3 AD8066, IC4 AD8066, IC5 LT1713, IC6 LT1713, IC7 AD8066, X1 87437-0443, X2 87437-0443, X3 87437-0443

Commit message: Removed guard ring due to ocurring shorts and adjusted supply rail resistors
Parts:
- R20, R21, R23, R24, R28, R29, R32, R33, R36, R40, R41, R44, R45: value 75 -> 1
Changed lines of the file:
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@@
 <?xml version="1.0" encoding="utf-8"?>
 <!DOCTYPE eagle SYSTEM "eagle.dtd">
-<eagle version="9.5.1">
+<eagle version="9.5.2">
 <drawing>
 <settings>
@@
 <attribute name="SPICEPREFIX" value="R" x="17.526" y="47.498" size="1.778" layer="27" rot="R90" display="off"/>
 </element>
-<element name="R20" library="rcl" library_urn="urn:adsk.eagle:library:334" package="R0603" package3d_urn="urn:adsk.eagle:package:23555/2" value="75" x="18.542" y="50.546" smashed="yes" rot="R180">
+<element name="R20" library="rcl" library_urn="urn:adsk.eagle:library:334" package="R0603" package3d_urn="urn:adsk.eagle:package:23555/2" value="1" x="18.542" y="50.546" smashed="yes" rot="R180">
 <attribute name="NAME" x="17.272" y="51.054" size="1.016" layer="26" font="vector" ratio="20" rot="MR180"/>
 <attribute name="SPICEPREFIX" value="R" x="18.542" y="50.546" size="1.778" layer="27" rot="R180" display="off"/>
 </element>
-<element name="R21" library="rcl" library_urn="urn:adsk.eagle:library:334" package="R0603" package3d_urn="urn:adsk.eagle:package:23555/2" value="75" x="9.398" y="42.926" smashed="yes" rot="R180">
+<element name="R21" library="rcl" library_urn="urn:adsk.eagle:library:334" package="R0603" package3d_urn="urn:adsk.eagle:package:23555/2" value="1" x="9.398" y="42.926" smashed="yes" rot="R180">
 <attribute name="NAME" x="6.858" y="41.148" size="1.016" layer="25" font="vector" ratio="20"/>
 <attribute name="SPICEPREFIX" value="R" x="9.398" y="42.926" size="1.778" layer="27" rot="R180" display="off"/>
@@
 <attribute name="SPICEPREFIX" value="R" x="21.59" y="49.276" size="1.778" layer="27" rot="R90" display="off"/>
 </element>
-<element name="R23" library="rcl" library_urn="urn:adsk.eagle:library:334" package="R0603" package3d_urn="urn:adsk.eagle:package:23555/2" value="75" x="28.194" y="54.61" smashed="yes">
+<element name="R23" library="rcl" library_urn="urn:adsk.eagle:library:334" package="R0603" package3d_urn="urn:adsk.eagle:package:23555/2" value="1" x="28.194" y="54.61" smashed="yes">
 <attribute name="NAME" x="26.924" y="55.372" size="1.016" layer="25" font="vector" ratio="20"/>
 <attribute name="SPICEPREFIX" value="R" x="28.194" y="54.61" size="1.778" layer="27" display="off"/>
 </element>
-<element name="R24" library="rcl" library_urn="urn:adsk.eagle:library:334" package="R0603" package3d_urn="urn:adsk.eagle:package:23555/2" value="75" x="28.194" y="42.926" smashed="yes">
+<element name="R24" library="rcl" library_urn="urn:adsk.eagle:library:334" package="R0603" package3d_urn="urn:adsk.eagle:package:23555/2" value="1" x="28.194" y="42.926" smashed="yes">
 <attribute name="NAME" x="29.591" y="39.751" size="1.016" layer="25" font="vector" ratio="20" rot="R90"/>
 <attribute name="SPICEPREFIX" value="R" x="28.194" y="42.926" size="1.778" layer="27" display="off"/>
@@
 <attribute name="SPICEPREFIX" value="R" x="9.398" y="46.99" size="1.778" layer="27" display="off"/>
 </element>
-<element name="R28" library="rcl" library_urn="urn:adsk.eagle:library:334" package="R0603" package3d_urn="urn:adsk.eagle:package:23555/2" value="75" x="39.878" y="50.292" smashed="yes" rot="R90">
+<element name="R28" library="rcl" library_urn="urn:adsk.eagle:library:334" package="R0603" package3d_urn="urn:adsk.eagle:package:23555/2" value="1" x="39.878" y="50.292" smashed="yes" rot="R90">
 <attribute name="NAME" x="39.37" y="49.149" size="1.016" layer="26" font="vector" ratio="20" rot="MR90"/>
 <attribute name="SPICEPREFIX" value="R" x="39.878" y="50.292" size="1.778" layer="27" rot="R90" display="off"/>
 </element>
-<element name="R29" library="rcl" library_urn="urn:adsk.eagle:library:334" package="R0603" package3d_urn="urn:adsk.eagle:package:23555/2" value="75" x="45.72" y="42.672" smashed="yes">
+<element name="R29" library="rcl" library_urn="urn:adsk.eagle:library:334" package="R0603" package3d_urn="urn:adsk.eagle:package:23555/2" value="1" x="45.72" y="42.672" smashed="yes">
 <attribute name="NAME" x="45.72" y="40.894" size="1.016" layer="25" font="vector" ratio="20"/>
 <attribute name="SPICEPREFIX" value="R" x="45.72" y="42.672" size="1.778" layer="27" display="off"/>
@@
 <attribute name="SPICEPREFIX" value="R" x="25.654" y="49.276" size="1.778" layer="27" rot="R90" display="off"/>
 </element>
-<element name="R32" library="rcl" library_urn="urn:adsk.eagle:library:334" package="R0603" package3d_urn="urn:adsk.eagle:package:23555/2" value="75" x="15.24" y="66.802" smashed="yes">
+<element name="R32" library="rcl" library_urn="urn:adsk.eagle:library:334" package="R0603" package3d_urn="urn:adsk.eagle:package:23555/2" value="1" x="15.24" y="66.802" smashed="yes">
 <attribute name="NAME" x="16.51" y="67.564" size="1.016" layer="25" font="vector" ratio="20" rot="R90"/>
 <attribute name="SPICEPREFIX" value="R" x="15.24" y="66.802" size="1.778" layer="27" display="off"/>
 </element>
-<element name="R33" library="rcl" library_urn="urn:adsk.eagle:library:334" package="R0603" package3d_urn="urn:adsk.eagle:package:23555/2" value="75" x="12.192" y="57.15" smashed="yes">
+<element name="R33" library="rcl" library_urn="urn:adsk.eagle:library:334" package="R0603" package3d_urn="urn:adsk.eagle:package:23555/2" value="1" x="12.192" y="57.15" smashed="yes">
 <attribute name="NAME" x="11.684" y="55.372" size="1.016" layer="25" font="vector" ratio="20"/>
 <attribute name="SPICEPREFIX" value="R" x="12.192" y="57.15" size="1.778" layer="27" display="off"/>
@@
 <attribute name="SPICEPREFIX" value="R" x="9.652" y="63.5" size="1.778" layer="27" rot="R90" display="off"/>
 </element>
-<element name="R36" library="rcl" library_urn="urn:adsk.eagle:library:334" package="R0603" package3d_urn="urn:adsk.eagle:package:23555/2" value="75" x="54.864" y="50.8" smashed="yes" rot="R180">
+<element name="R36" library="rcl" library_urn="urn:adsk.eagle:library:334" package="R0603" package3d_urn="urn:adsk.eagle:package:23555/2" value="1" x="54.864" y="50.8" smashed="yes" rot="R180">
 <attribute name="NAME" x="57.404" y="49.53" size="1.016" layer="25" font="vector" ratio="20" rot="R90"/>
 <attribute name="SPICEPREFIX" value="R" x="54.864" y="50.8" size="1.778" layer="27" rot="R180" display="off"/>
@@
 <attribute name="SPICEPREFIX" value="R" x="12.192" y="66.802" size="1.778" layer="27" display="off"/>
 </element>
-<element name="R40" library="rcl" library_urn="urn:adsk.eagle:library:334" package="R0603" package3d_urn="urn:adsk.eagle:package:23555/2" value="75" x="44.196" y="66.802" smashed="yes">
+<element name="R40" library="rcl" library_urn="urn:adsk.eagle:library:334" package="R0603" package3d_urn="urn:adsk.eagle:package:23555/2" value="1" x="44.196" y="66.802" smashed="yes">
 <attribute name="NAME" x="45.593" y="66.294" size="1.016" layer="26" font="vector" ratio="20" rot="MR0"/>
 <attribute name="SPICEPREFIX" value="R" x="44.196" y="66.802" size="1.778" layer="27" display="off"/>
 </element>
-<element name="R41" library="rcl" library_urn="urn:adsk.eagle:library:334" package="R0603" package3d_urn="urn:adsk.eagle:package:23555/2" value="75" x="47.244" y="59.182" smashed="yes">
+<element name="R41" library="rcl" library_urn="urn:adsk.eagle:library:334" package="R0603" package3d_urn="urn:adsk.eagle:package:23555/2" value="1" x="47.244" y="59.182" smashed="yes">
 <attribute name="NAME" x="45.974" y="59.69" size="1.016" layer="26" font="vector" ratio="20" rot="MR180"/>
 <attribute name="SPICEPREFIX" value="R" x="47.244" y="59.182" size="1.778" layer="27" display="off"/>
@@
 <attribute name="SPICEPREFIX" value="R" x="19.558" y="61.976" size="1.778" layer="27" rot="R90" display="off"/>
 </element>
-<element name="R44" library="rcl" library_urn="urn:adsk.eagle:library:334" package="R0603" package3d_urn="urn:adsk.eagle:package:23555/2" value="75" x="28.194" y="66.802" smashed="yes" rot="R180">
+<element name="R44" library="rcl" library_urn="urn:adsk.eagle:library:334" package="R0603" package3d_urn="urn:adsk.eagle:package:23555/2" value="1" x="28.194" y="66.802" smashed="yes" rot="R180">
 <attribute name="NAME" x="29.718" y="66.675" size="1.016" layer="25" font="vector" ratio="20"/>
 <attribute name="SPICEPREFIX" value="R" x="28.194" y="66.802" size="1.778" layer="27" rot="R180" display="off"/>
 </element>
-<element name="R45" library="rcl" library_urn="urn:adsk.eagle:library:334" package="R0603" package3d_urn="urn:adsk.eagle:package:23555/2" value="75" x="28.194" y="57.15" smashed="yes">
+<element name="R45" library="rcl" library_urn="urn:adsk.eagle:library:334" package="R0603" package3d_urn="urn:adsk.eagle:package:23555/2" value="1" x="28.194" y="57.15" smashed="yes">
 <attribute name="NAME" x="24.257" y="57.404" size="1.016" layer="25" font="vector" ratio="20"/>
 <attribute name="SPICEPREFIX" value="R" x="28.194" y="57.15" size="1.778" layer="27" display="off"/>
